File: PCB/The_Ping_Ting/filter3.kicad_sch (KiCad schematic)
At the start: 18 parts, among them SW401 SW_SP3T, U106 LM324

Commit message: REVV 1.2 - Updated resonance feedback resistance Updated the feedback resistance in the mid and high frequency feedback circuit to get a more "stable" resonance level.
Parts:
- R410: value 100 -> 100R
Other:
- company: (none) -> Kromftronics
- title: (none) -> Low Frequency Filter
Changed lines of the file:
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@@
 	(generator_version "8.0")
 	(paper "A4")
+	(title_block
+		(title "Low Frequency Filter")
+		(date "2024-09-07")
+		(rev "1.2")
+		(company "Kromftronics")
+	)
 	(junction
 		(at 144.78 93.98)
@@
 			)
 		)
-		(property "Value" "100"
+		(property "Value" "100R"
 			(at 114.3 111.3536 90)
 			(effects
